File: hardware/esc/esc/single_esc_1.kicad_sch (KiCad schematic)
At the start: 36 parts, among them Q1 Q_NMOS, Q2 Q_NMOS, Q3 Q_NMOS, Q4 Q_NMOS, Q5 Q_NMOS, Q6 Q_NMOS, U1 NSG2065Q, U2 AT32F421G8U7

Commit message: Routing done!
Parts:
- removed D1: LED, LED_SMD:LED_0603_1608Metric, symbol Device:LED
- removed R20: 2.2k, Resistor_SMD:R_0402_1005Metric, symbol Device:R
- renumbered R15 to R10, R22 to R10, R19 to R9, R10 to R9, R18 to R9
Connections:
- net B: now also R9.4; no longer R9.2
- net BEMF_A: now also R9.5; no longer R9.2
- net BEMF_B: now also R9.3, R9.7; no longer R9.1, R9.2
- net BEMF_C: now also R10.4; no longer R10.1
- net BEMF_COM: now also R9.6, R9.8; no longer R9.1, R9.1
- net C: now also R10.3; no longer R10.2
Other:
- moved on the sheet: R10B, R9C, R9D
