File: hardware/esc/esc/single_esc_2.kicad_sch (KiCad schematic)
At the start: 36 parts, among them Q10 Q_NMOS, Q11 Q_NMOS, Q12 Q_NMOS, Q7 Q_NMOS, Q8 Q_NMOS, Q9 Q_NMOS, U4 AT32F421G8U7, U5 NSG2065Q

Commit message: Routing done!
Parts:
- removed D2: LED, LED_SMD:LED_0603_1608Metric, symbol Device:LED
- removed R24: 2.2k, Resistor_SMD:R_0402_1005Metric, symbol Device:R
- renumbered R19 to R15, R22 to R15, R10 to R15, R9 to R19, R18 to R19
Connections:
- net A: now also R19.8; no longer R19.4
- net B: now also R15.6; no longer R15.4
- net BEMF_A: now also R19.6, R19.7; no longer R19.3, R19.4
- net BEMF_B: now also R15.2, R15.5; no longer R15.3, R15.4
- net BEMF_C: now also R15.7; no longer R15.3
- net BEMF_COM: now also R15.1, R19.5; no longer R15.3, R19.3
- net C: now also R15.8; no longer R15.4
