File: hardware/esc/esc/single_esc_4.kicad_sch (KiCad schematic)
At the start: 36 parts, among them Q19 Q_NMOS, Q20 Q_NMOS, Q21 Q_NMOS, Q22 Q_NMOS, Q23 Q_NMOS, Q24 Q_NMOS, U8 AT32F421G8U7, U9 NSG2065Q

Commit message: Routing done!
Parts:
- removed D4: LED, LED_SMD:LED_0603_1608Metric, symbol Device:LED
- removed R64: 2.2k, Resistor_SMD:R_0402_1005Metric, symbol Device:R
- renumbered R9 to R19, R18 to R19, R15 to R22, R10 to R22, R19 to R22
Connections:
- net A: now also R19.4; no longer R19.8
- net B: now also R22.4; no longer R22.8
- net BEMF_A: now also R19.1, R19.3; no longer R19.7, R19.8
- net BEMF_B: now also R22.3; no longer R22.7
- net BEMF_C: now also R22.1, R22.6; no longer R22.7, R22.8
- net BEMF_COM: now also R19.2, R22.5; no longer R19.7, R22.7
- net C: now also R22.2; no longer R22.8
Other:
- moved on the sheet: R19A
