File: hardware/fc/fc/fc.kicad_sch (KiCad schematic)
At the start: 24 parts, among them J1 Camera, J2 ELRS, J3 Buzzer, J4 MMCX (Antenna), SW1 DIPx03, U1 STM32F405RGTx, U2 ICM-42688-P, U3 max7456eui+, U4 a, U5 BL8072CLTR50

Commit message: More work on FC
Parts:
- removed U5: BL8072CLTR50, symbol BL8072:BL8072
- added C13, C14, C15, C16: 1uF, symbol Device:C
- added C17, C18: 22nF, symbol Device:C
- added C19, C20: 100nF, symbol Device:C_Small
- added C21: 100nF, symbol Device:C
- added C22, C27: 180uF 35V, symbol Device:C_Polarized_Small_US
- added C23, C26: 1uF, symbol Device:C_Small
- added C24, C25: 470uF 35V, symbol Device:C_Polarized_Small_US
- added C28, C29: 2.2uF, symbol Device:C_Small
- added D1, D2: LED, symbol Device:LED
- added D3, D4: D_Schottky, symbol Device:D_Schottky
- added D5, D6: 1N5820, symbol Device:D_Schottky_Small
- added F1: 5A Fuse, symbol Device:Fuse
- added J5: ESC, symbol Connector_Generic:Conn_01x08
- added J6: USB_B_Micro, symbol Connector:USB_B_Micro
- added L1, L2: 68uH/2A, symbol Device:L
- added Q1: Q_PMOS, symbol Device:Q_PMOS
- added R10: 1.8k, symbol Device:R
- added R11: 1.1k, symbol Device:R
- added R12, R13: 2.2K, symbol Device:R
- added R3: 10k, symbol Device:R_Small
- added R4: 100k, symbol Device:R_Small
- added R5, R6: 75, symbol Device:R
- added R7, R8: 22, symbol Device:R_Small
- added R9: R, symbol Device:R
- added U10: BMP280, Package_LGA:Bosch_LGA-8_2x2.5mm_P0.65mm_ClockwisePinNumbering, symbol Sensor_Pressure:BMP280
- added U5: XL1509-ADJ, Package_SO:SOIC-8_3.9x4.9mm_P1.27mm, symbol Regulator_Switching:XL1509-ADJ
- added U6: BL8072CLTR33, symbol BL8072:BL8072
- added U7: SGM2212-3.3XKC3G/TR, SOT-223-3_SGM2212_SNC, symbol SGM2212-3-3XKC3G-TR:SGM2212-3.3XKC3G_TR
- added U8: W25Q128JVSIQ TR, SOIC_208MIL_WIN, symbol W25Q128JVSIQ:W25Q128JVSIQ_TR
- added U9: XL1509-5.0, Package_SO:SOIC-8_3.9x4.9mm_P1.27mm, symbol Regulator_Switching:XL1509-5.0
- added Y1: 27MHz, symbol Device:Crystal_GND24_Small
- added Y2: CSTNE8M00G520000R0, CSTNE8M00G520000R0:OSC_CSTNE8M00G520000R0, symbol CSTNE8M00G520000R0:CSTNE8M00G520000R0
- C1, C2: value 1uF -> 100nF
Connections:
- net IMU_INT2 is gone; now on net IMU_CLKIN: U2.9 (INT2/FSYNC/CLKIN)
- net IMU_SDIO is gone; now on net IMU_SDI: U2.14 (AP_SDA/AP_SDIO/AP_SDI)
- net +3.3V: now also C1.1, C2.1, U1.1 (VBAT), U1.13 (VDDA), U1.19 (VDD), U1.32 (VDD), U1.48 (VDD), U1.64 (VDD), C14.1, C21.1, R12.1, R13.1, U10.2 (CSB), U10.6 (VDDIO), U10.8 (VDD), U6.2 (Vout), U8.3 (/WP(IO2)), U8.7 (/HOLD_/RESET), U8.8 (VCC)
- net +5V: now also J2.3 (Pin_3), C22.1, D3.2 (A), L1.2, U9.3 (FB); no longer C2.1
- net GND: now also J2.4 (Pin_4), J3.2 (Pin_2), U1.12 (VSSA), U1.18 (VSS), U1.63 (VSS), C13.2, C14.2, C15.2, C16.2, C17.2, C18.2, C19.2, C20.2, C21.2, C22.2, C23.2, C24.2, C25.2, C26.2, C27.2, C28.2, C29.2, D5.2 (A), D6.2 (A), J5.2 (Pin_2), J6.5 (GND), J6.SH (Shield), R11.2, R3.2, R5.2, R6.2, R9.2, U10.1 (GND), U10.5 (SDO), U10.7 (GND), U5.4 (~{EN}), U5.5 (GND), U5.6 (GND), U5.7 (GND), U5.8 (GND), U6.1 (Vss), U7.1 (GND), U8.4 (GND), U9.4 (~{EN}), U9.5 (GND), U9.6 (GND), U9.7 (GND), U9.8 (GND), Y1.2 (G), Y1.4 (G), Y2.2
- net IMU_3.3V: now also C16.1, C17.1, C18.1, U7.2 (VOUT)
- net IMU_CS: now also U1.20 (PA4)
- net IMU_INT1: now also U1.24 (PC4)
- net IMU_SCLK: now also U1.21 (PA5)
- net IMU_SDO: now also U1.23 (PA7)
- net OSD CS: now also U1.50 (PA15)
- net OSD SCLK: now also U1.51 (PC10)
- net OSD SDIN: now also U1.52 (PC11)
- net OSD SDOUT: now also U1.57 (PB5)
- net VBAT: now also F1.1; no longer C1.1
- net CURRENT: now reaches U1.10 (PC2)
- net CURRENT: now also C19.1, J5.3 (Pin_3)
- net BEEPER: now reaches U1.2 (PC13)
- net BEEPER: now also J3.1 (Pin_1)
- net IMU_SDI: now reaches U1.22 (PA6)
- net I2C_SCL: now reaches U1.29 (PB10)
- net I2C_SCL: now also R12.2, U10.4 (SCK)
- net LED1_STATUS: now reaches U1.3 (PC14)
- net LED1_STATUS: now also D2.2 (A)
- net I2C_SDA: now reaches U1.30 (PB11)
- net I2C_SDA: now also R13.2, U10.3 (SDI)
- net at U1.31 (VCAP_1): now also C29.1
- net FLASH_CS: now reaches U1.33 (PB12)
- net FLASH_CS: now also U8.1 (/CS)
- net SPI2_SCK: now reaches U1.34 (PB13)
- net SPI2_SCK: now also U8.6 (CLK)
- net SPI2_DI: now reaches U1.35 (PB14)
- net SPI2_DI: now also U8.5 (DI(IO0))
- net SPI2_DO: now reaches U1.36 (PB15)
- net SPI2_DO: now also U8.2 (DO(IO1))
- net MOTOR_4: now reaches U1.39 (PC8)
- net MOTOR_4: now also J5.8 (Pin_8)
- net LED0_STATUS: now reaches U1.4 (PC15)
- net LED0_STATUS: now also D1.2 (A)
- net MOTOR_3: now reaches U1.40 (PC9)
- net MOTOR_3: now also J5.7 (Pin_7)
- net MOTOR_2: now reaches U1.41 (PA8)
- net MOTOR_2: now also J5.6 (Pin_6)
- net MOTOR_1: now reaches U1.42 (PA9)
- net MOTOR_1: now also J5.5 (Pin_5)
- net USB_D-: now reaches U1.44 (PA11)
- net USB_D-: now also R8.2
- net USB_D+: now reaches U1.45 (PA12)
- net USB_D+: now also R7.2
- net at U1.47 (VCAP_2): now also C28.1
- net OSC_IN: now reaches U1.5 (PH0)
- net OSC_IN: now also Y2.1
- net UART1_TX: now reaches U1.58 (PB6)
- net UART1_TX: now also J2.2 (Pin_2)
- net UART1_RX: now reaches U1.59 (PB7)
- net UART1_RX: now also J2.1 (Pin_1)
- net OSC_OUT: now reaches U1.6 (PH1)
- net OSC_OUT: now also Y2.3
- net BOOT0: now reaches U1.60 (BOOT0)
- net IMU_CLKIN: now reaches U1.61 (PB8)
- net at U1.9 (PC1): now also C20.1, R3.1, R4.2
- net at U3.5 (CLKIN): now also Y1.3
- net at U3.6 (XFB): now also Y1.1
- new net: D2.1 (K), R5.1
- new net: R10.1, R11.1, U5.3 (FB)
- new net: F1.2, Q1.D
- new net: Q1.G, R9.1
- new net: D1.1 (K), R6.1
- new net: J6.3 (D+), R7.1
- new net: J6.2 (D-), R8.1
- new net: D6.1 (K), L2.1, U5.2 (OUT)
- new net: D5.1 (K), L1.1, U9.2 (OUT)
- new net +4.5V: C13.1, C15.1, D3.1 (K), D4.1 (K), U6.3 (Vin), U7.3 (VIN)
- new net +BATT: J5.1 (Pin_1), R4.1
- new net VBUS: D4.2 (A), J6.1 (VBUS)
- new net VIN: C23.1, C24.1, C25.1, C26.1, Q1.S, U5.1 (VIN), U9.1 (VIN)
- new net VTX_5V: C27.1, L2.2, R10.2
- no-connect marks 3 -> 10
Other:
- note added: "3.3V"
- note added: "3.3V LDO"
- note added: "3.3V LDO - IMU"
- note added: "4.5V"
- note added: "5V BEC"
- note added: "8MHz"
- note added: "Baro"
- note added: "Buzzer"
- note added: "Flash (Blackbox)"
- note added: "IMU"
- note added: "LEDs"
- note added: "OSD"
- note added: "Reverse Polarity Protection"
- note added: "VTX"
- note added: "VTX 3.3V BEC"
- moved on the sheet: C10, C11, C12, C3, C4, C5, C6, C7, C8, C9, J1, J2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
